Commit message: [1] Added realistic 3D model of GoPiGo3. [2] Included key_teleop package for teleoperation with the keyboard

File: gopigo3_description/urdf/common_properties.xacro (robot description, xacro)
@@ -1,7 +1,9 @@
 <?xml version="1.0" ?>
 <robot name="xacro_properties" xmlns:xacro="http://ros.org/wiki/xacro">
+<xacro:property name="black_opacity" value="0.5" />
+<xacro:property name="blue_opacity" value="1.0" />
   <!-- Init colour -->
   <material name="black">
-      <color rgba="0.0 0.0 0.0 1.0"/>
+      <color rgba="0.0 0.0 0.0 ${black_opacity}"/>
   </material>
   <material name="dark">
@@ -12,5 +14,11 @@
   </material>
   <material name="blue">
-    <color rgba="0.0 0.0 0.8 1.0"/>
+    <color rgba="0.0 0.0 0.8 ${blue_opacity}"/>
+  </material>
+  <material name="cyan">
+    <color rgba="0.0 1.0 1.0 1.0"/>
+  </material>
+  <material name="yellow">
+    <color rgba="1.0 1.0 0.0 1.0"/>
   </material>
   <material name="green">

File: gopigo3_description/urdf/gopigo3.gazebo.xacro (robot description, xacro)
@@ -3,4 +3,6 @@
   <xacro:arg name="laser_visual" default="false"/>
   <xacro:arg name="imu_visual"   default="false"/>
+  <xacro:arg name="camera_visual"   default="false"/>
+  <xacro:arg name="distance_visual" default="false"/>
   <gazebo reference="base_link">
     <material>Gazebo/DarkGrey</material>
@@ -54,14 +56,50 @@
       <leftJoint>wheel_left_joint</leftJoint>
       <rightJoint>wheel_right_joint</rightJoint>
-      <!--wheelSeparation>0.160</wheelSeparation>
-      <wheelDiameter>0.066</wheelDiameter-->
-      <wheelSeparation>0.115</wheelSeparation>
-      <wheelDiameter>0.065</wheelDiameter>
+      <wheelSeparation>0.116</wheelSeparation>
+      <wheelDiameter>0.066</wheelDiameter>
       <wheelAcceleration>1</wheelAcceleration>
-      <wheelTorque>10</wheelTorque>
+      <wheelTorque>5</wheelTorque>
       <rosDebugLevel>na</rosDebugLevel>
     </plugin>
   </gazebo>
-<!-- IMU sensor active -->
+<!-- Distance Sensor controller -->
+  <gazebo reference="distance_sensor">
+    <sensor type="ray" name="laser_distance">
+      <pose>0 0 0 0 0 0</pose>
+      <visualize>true</visualize>
+      <update_rate>10</update_rate>
+      <ray>
+         <scan>
+            <horizontal>
+               <samples>10</samples>
+               <resolution>1</resolution>
+               <min_angle>-0.01</min_angle>
+               <max_angle>0.01</max_angle>
+            </horizontal>
+            <vertical>
+               <samples>10</samples>
+               <resolution>1</resolution>
+               <min_angle>-0.01</min_angle>
+               <max_angle>0.01</max_angle>
+            </vertical>
+         </scan>
+         <range>
+            <min>0.01</min>
+            <max>3</max>
+            <resolution>0.01</resolution>
+         </range>
+      </ray>
+      <plugin filename="libgazebo_ros_range.so" name="gazebo_ros_ir">
+         <gaussianNoise>0.005</gaussianNoise>
+         <alwaysOn>true</alwaysOn>
+         <updateRate>0.0</updateRate>
+         <topicName>gopigo/distance</topicName>
+         <frameName>distance_sensor</frameName>
+         <radiation>INFRARED</radiation>
+         <fov>0.02</fov>
+      </plugin>
+    </sensor>
+   </gazebo>
+<!-- IMU sensor -->
   <gazebo reference="imu_link">
     <sensor type="imu" name="imu">
@@ -120,5 +158,4 @@
         <range>
           <min>0.120</min>
-          <!--max>3.5</max-->
           <max>10</max>
           <resolution>0.015</resolution>
@@ -126,6 +163,9 @@
         <noise>
           <type>gaussian</type>
+          <!-- Noise parameters based on published spec for YDLIDAR X4
+               is 1.5% at half range 4m (= 60mm, "+-160mm" accuracy at max. range 8m).
+               A mean of 0.0m and stddev of 0.020m will put 99.7% of samples
+               within 0.16m of the true reading. -->
           <mean>0.0</mean>
-          <!--stddev>0.01</stddev-->
           <stddev>0.02</stddev>
         </noise>
@@ -141,5 +181,5 @@
     <sensor type="ray" name="laser_distance">
       <pose>0 0 0 0 0 0</pose>
-      <visualize>true</visualize>
+      <visualize>$(arg distance_visual)</visualize>
       <update_rate>10</update_rate>
       <ray>
@@ -178,5 +218,6 @@
   <gazebo reference="camera">
     <sensor type="camera" name="camera1">
-      <update_rate>30.0</update_rate>
+      <always_on>true</always_on>
+      <visualize>$(arg camera_visual)</visualize>
       <camera name="front">
         <horizontal_fov>1.3962634</horizontal_fov>
@@ -193,5 +234,5 @@
       <plugin name="camera_controller" filename="libgazebo_ros_camera.so">
         <alwaysOn>true</alwaysOn>
-        <updateRate>0.0</updateRate>
+        <updateRate>30.0</updateRate>
         <cameraName>gopigo/camera1</cameraName>
         <imageTopicName>image_raw</imageTopicName>

File: gopigo3_description/urdf/gopigo3.urdf.xacro (robot description, xacro)
@@ -1,129 +1,133 @@
 <?xml version="1.0" ?>
-<robot name="gopigo3_sim" xmlns:xacro="http://ros.org/wiki/xacro">
+<robot name="gopigo3" xmlns:xacro="http://ros.org/wiki/xacro">
   <xacro:include filename="$(find gopigo3_description)/urdf/common_properties.xacro"/>
   <xacro:include filename="$(find gopigo3_description)/urdf/gopigo3.gazebo.xacro"/>
-<!-- Base Footprint Link (base_footprint) -->
+  <xacro:property name="CADscale" value="0.0012" />
+  <!-- Which sensors to include -->
+<xacro:arg name="imu" default="false" />
+<!--xacro:property name="imu" value="true"/-->
+<xacro:arg name="distance"        default="true"/>
+<xacro:arg name="pi_camera"       default="true"/>
+<xacro:arg name="lds"             default="true"/>
+<!-- ============ 'base_footprint' is the ground link ===================== -->
   <link name="base_footprint"/>
-<!-- JOINT base_link to base_footprint-->
   <joint name="base_joint" type="fixed">
     <parent link="base_footprint"/>
     <child link="base_link"/>
-    <!--origin xyz="0.0 0.0 0.010" rpy="0 0 0"/-->
-    <origin xyz="0 0 0.0875" rpy="0 0 0"/>
-  </joint>
-<!-- Base Link (base_link) -->
+    <!-- base_link is placed at the center of gravity of GoPiGo3 body -->
+    <origin xyz="0 0 0.075" rpy="0 0 0"/>
+  </joint>
+<!-- ============ 'base_link' simulates GoPiGo3 body mass and moment of inertia
+                   and act as the robot reference frame =================== -->
   <link name="base_link">
+  <!-- **** 'base_link' COLLISION & INERTIA **** -->
+    <collision>
+      <origin xyz="-0.032 0 0.070" rpy="0 0 0"/>
+      <geometry>
+        <box size="0.21 0.105 0.11"/>
+      </geometry>
+    </collision>
+    <inertial>
+      <origin xyz="0 0 0" rpy="0 0 0"/>
+      <mass value="0.534"/>
+      <inertia ixx="1.03e-03" ixy="-1.54e-03" ixz="-2.94e-03"
+               iyy="2.50e-03" iyz="-3.08e-03"
+               izz="2.45e-03" />
+    </inertial>
+  </link>
+<!-- ============  'base_link_cad' is the solid model of robot body ====== -->
+  <joint name="base_joint_cad" type="fixed">
+    <parent link="base_footprint"/>
+    <child link="base_link_cad"/>
+    <!-- CAD of body of GoPiGo3 has its reference coordinate system at the center of the wheels shaft -->
+    <origin xyz="0 0 0.033" rpy="0 0 -4.71"/>
+  </joint>
+  <link name="base_link_cad">
     <visual>
-      <!--origin xyz="-0.032 0 0.0" rpy="0 0 0"/-->
-      <origin xyz="0 0 0" rpy="0 0 0"/>
-      <geometry>
-        <!--mesh filename="package://turtlebot3_description/meshes/bases/burger_base.stl" scale="0.001 0.001 0.001"/-->
-        <box size="0.25 0.25 0.125"/>
-      </geometry>
-      <material name="light_black"/>
+      <!-- Decentering of the CAD model coordinate system-->
+      <origin xyz="0.024 0.097 -0.038" rpy="0 0 0"/>
+      <geometry>
+        <mesh filename="package://gopigo3_description/meshes/GoPiGo3_Body.stl" scale="${CADscale} ${CADscale} ${CADscale}"/>
+      </geometry>
+      <material name="blue"/>
     </visual>
-    <collision>
-      <origin xyz="-0.032 0 0.070" rpy="0 0 0"/>
-      <geometry>
-        <!--box size="0.140 0.140 0.143"/-->
-        <box size="0.25 0.25 0.125"/>
-      </geometry>
-    </collision>
-    <inertial>
-      <origin xyz="0 0 0" rpy="0 0 0"/>
-      <mass value="8.2573504e-01"/>
-      <inertia ixx="2.2124416e-03" ixy="-1.2294101e-05" ixz="3.4938785e-05"
-               iyy="2.1193702e-03" iyz="-5.0120904e-06"
-               izz="2.0064271e-03" />
-    </inertial>
-  </link>
-<!-- JOINT wheel_left_link to base_link -->
+  </link>
+<!-- ============ wheel_left ====================== -->
   <joint name="wheel_left_joint" type="continuous">
     <parent link="base_link"/>
     <child link="wheel_left_link"/>
-    <!--origin xyz="0.0 0.08 0.023" rpy="-1.57 0 0"/>
-    <axis xyz="0 0 1"/-->
-    <origin xyz="0.1 0.15 0.0125" rpy="0 0 0" />
-    <axis xyz="0 1 0"/>
-  </joint>
-<!-- Left Wheel link (wheel_left_link) -->
+    <!-- Ty is half the shaft lenght -->
+    <!-- Tz = -(0.075 base_link cdg -0.033 wheel radius) = -0.042 -->
+    <origin xyz="0 0.058 -0.042" rpy="0 0 1.57"/>
+    <axis xyz="-1 0 0"/>
+  </joint>
   <link name="wheel_left_link">
     <visual>
-      <origin xyz="0 0 0" rpy="1.57 0 0"/>
-      <geometry>
-        <!--mesh filename="package://turtlebot3_description/meshes/wheels/left_tire.stl" scale="0.001 0.001 0.001"/-->
-        <cylinder length="0.05" radius="0.1" />
-      </geometry>
-      <material name="dark"/>
+      <!-- Decentering of wheel CAD model coordinate system-->
+      <origin xyz="-0.195 -0.173 -0.029" rpy="0 0 0"/>
+      <geometry>
+        <mesh filename="package://gopigo3_description/meshes/GoPiGo3_Wheel.stl" scale="0.001 0.001 0.001"/>
+      </geometry>
+      <material name="black"/>
     </visual>
+  <!-- **** 'wheel_left' COLLISION & INERTIA **** -->
     <collision>
       <origin xyz="0 0 0" rpy="0 0 0"/>
       <geometry>
-        <!--cylinder length="0.018" radius="0.033"/-->
-        <cylinder length="0.05" radius="0.1" />
+        <cylinder length="0.026" radius="0.033"/>
       </geometry>
     </collision>
     <inertial>
       <origin xyz="0 0 0" />
-      <mass value="2.8498940e-02" />
-      <inertia ixx="1.1175580e-05" ixy="-4.2369783e-11" ixz="-5.9381719e-09"
-               iyy="1.1192413e-05" iyz="-1.4400107e-11"
-               izz="2.0712558e-05" />
-      </inertial>
-  </link>
-<!-- JOINT wheel_right_link to base_link -->
+      <mass value="0.032" />
+      <inertia ixx="1.74e-05" ixy="0" ixz="0"
+               iyy="1.05e-05" iyz="0"
+               izz="1.05e-05" />
+    </inertial>
+  </link>
+<!-- ============ wheel_right ====================== -->
   <joint name="wheel_right_joint" type="continuous">
     <parent link="base_link"/>
     <child link="wheel_right_link"/>
-    <!--origin xyz="0.0 -0.080 0.023" rpy="-1.57 0 0"/>
-    <axis xyz="0 0 1"/-->
-    <origin xyz="0.1 -0.15 0.0125" rpy="0 0 0" />
-    <axis xyz="0 1 0" />
-  </joint>
-<!-- Right Wheel -->
+    <origin xyz="0 -0.058 -0.042" rpy="0 0 -1.57"/>
+    <!--axis xyz="0 0 1"/-->
+    <axis xyz="1 0 0"/>
+  </joint>
   <link name="wheel_right_link">
     <visual>
-      <origin xyz="0 0 0" rpy="1.57 0 0"/>
-      <geometry>
-        <!--mesh filename="package://turtlebot3_description/meshes/wheels/right_tire.stl" scale="0.001 0.001 0.001"/-->
-        <cylinder length="0.05" radius="0.1" />
-      </geometry>
-      <material name="dark"/>
+      <!-- Decentering of wheel CAD model coordinate system-->
+      <origin xyz="-0.195 -0.173 -0.029" rpy="0 0 0"/>
+      <geometry>
+        <mesh filename="package://gopigo3_description/meshes/GoPiGo3_Wheel.stl" scale="0.001 0.001 0.001"/>
+      </geometry>
+      <material name="black"/>
     </visual>
+  <!-- **** 'wheel_right' COLLISION & INERTIA **** -->
     <collision>
       <origin xyz="0 0 0" rpy="0 0 0"/>
       <geometry>
-        <!--cylinder length="0.018" radius="0.033"/-->
-        <cylinder length="0.05" radius="0.1" />
+        <cylinder length="0.026" radius="0.033"/>
       </geometry>
     </collision>
     <inertial>
       <origin xyz="0 0 0" />
-      <mass value="2.8498940e-02" />
-      <inertia ixx="1.1175580e-05" ixy="-4.2369783e-11" ixz="-5.9381719e-09"
-               iyy="1.1192413e-05" iyz="-1.4400107e-11"
-               izz="2.0712558e-05" />
-      </inertial>
-  </link>
-<!-- JOINT caster_back_link to base_link-->
+      <mass value="0.032" />
+      <inertia ixx="1.74e-05" ixy="0" ixz="0"
+               iyy="1.05e-05" iyz="0"
+               izz="1.05e-05" />
+    </inertial>
+  </link>
+<!-- ============ caster_back ====================== -->
   <joint name="caster_back_joint" type="fixed">
     <parent link="base_link"/>
     <child link="caster_back_link"/>
-    <!--origin xyz="-0.081 0 -0.004" rpy="-1.57 0 0"/-->
-    <origin xyz="-0.1 0 -0.0625" rpy="0 0 0" />
-  </joint>
-<!-- Caster link (caster_back_link)-->
+    <origin xyz="-0.115 0 -0.075" rpy="0 0 0"/>
+  </joint>
   <link name="caster_back_link">
-    <visual name="caster_visual">
+  <!-- **** COLLISION & INERTIA **** -->
+    <collision>
       <origin xyz="0 0.001 0" rpy="0 0 0"/>
       <geometry>
-        <sphere radius="0.025" />
-      </geometry>
-    </visual>
-    <collision>
-      <origin xyz="0 0.001 0" rpy="0 0 0"/>
-      <geometry>
-        <!--box size="0.030 0.009 0.020"/-->
-        <sphere radius="0.025" />
+        <box size="0.030 0.009 0.020"/>
       </geometry>
     </collision>
@@ -136,101 +140,128 @@
     </inertial>
   </link>
-<!-- JOINT  imu_link to base_link -->
-  <joint name="imu_joint" type="fixed">
-    <parent link="base_link"/>
-    <child link="imu_link"/>
-    <origin xyz="-0.032 0 0.068" rpy="0 0 0"/>
-  </joint>
-<!-- IMU Link (imu_link) -->
-  <link name="imu_link"/>
-<!-- JOINT base_scan to base_link -->
-  <joint name="scan_joint" type="fixed">
-    <parent link="base_link"/>
-    <child link="base_scan"/>
-    <!--origin xyz="-0.032 0 0.172" rpy="0 0 0"/-->
-    <origin xyz="0.01 0.05 0.125" rpy="0 0 -1.6"/>
-  </joint>
-<!-- Laser Distance Sensor (base_scan) -->
-  <link name="base_scan">
-    <visual>
-      <origin xyz="0 0 0.0" rpy="0 0 0"/>
-      <geometry>
-        <!--mesh filename="package://turtlebot3_description/meshes/sensors/lds.stl" scale="0.001 0.001 0.001"/-->
-        <mesh filename="package://gopigo3_description/meshes/X4.stl" scale="0.0015 0.0015 0.0015"/>
-      </geometry>
-      <material name="dark"/>
-    </visual>
-    <collision>
-      <!--origin xyz="0.015 0 -0.0065" rpy="0 0 0"/-->
-      <origin xyz="0 0 0" rpy="0 0 0"/>
-      <geometry>
-        <!--cylinder length="0.0315" radius="0.055"/-->
-        <cylinder length="0.01575" radius="0.0275"/>
-      </geometry>
-    </collision>
-    <inertial>
-      <mass value="0.114" />
-      <origin xyz="0 0 0" />
-      <inertia ixx="0.001" ixy="0.0" ixz="0.0"
-               iyy="0.001" iyz="0.0"
-               izz="0.001" />
-    </inertial>
-  </link>
-<!-- JOINT camera to base_link -->
-  <joint name="joint_camera" type="fixed">
-    <axis xyz="0 0 1" />
-    <origin xyz="0 0 0" rpy="0 0 0"/>
-    <parent link="base_link"/>
-    <child link="camera"/>
-  </joint>
-<!-- 2D Camera (camera) -->
-  <link name="camera">
-    <visual>
-      <origin xyz="0.125 0 0.025" rpy="0 1.570795 0" />
-      <geometry>
-          <mesh filename="package://gopigo3_description/meshes/piCamera.stl" scale="0.0025 0.0025 0.0025"/>
-      </geometry>
-      <material name="yellow"/>
-    </visual>
-    <collision>
-      <origin xyz="0.1375 0 0.025" rpy="0 -1.570795 0" />
-      <geometry>
-        <box size="0.075 0.075 0.025"/>
-      </geometry>
-    </collision>
-    <inertial>
-      <origin xyz="0.1375 0 0.025" rpy="0 -1.570795 0" />
-      <mass value="1e-3" />
-      <inertia ixx="1e-6" ixy="0" ixz="0" iyy="1e-6" iyz="0" izz="1e-6" />
-    </inertial>
-  </link>
-<!-- JOINT distance_sensor to base_link -->
-  <joint name="distance_sensor_joint" type="fixed">
-    <axis xyz="0 1 0" />
-    <origin rpy="0 0 0" xyz="0 0 0" />
-    <parent link="base_link"/>
-    <child link="distance_sensor"/>
-  </joint>
-<!-- Distance Sensor -->
-  <link name="distance_sensor">
-    <visual>
-      <origin xyz="0.1 0 0.0755" rpy="1.570795 0 1.570795" />
-      <geometry>
-        <mesh filename="package://gopigo3_description/meshes/IR_Sensor_Sharp_GP2Y_solid.stl" scale="0.0025 0.0025 0.0025"/>
-      </geometry>
-      <material name="red"/>
-    </visual>
-    <collision>
-      <origin xyz="0.1 0 0.0775" rpy="1.570795 0 1.570795" />
-      <geometry>
-        <box size="0.005 0.005 0.005"/>
-      </geometry>
-    </collision>
-    <inertial>
-      <origin xyz="0.1 0 0.0755" rpy="1.570795 0 1.570795" />
-      <mass value="1e-5" />
-      <origin xyz="0 0 0" rpy="0 0 0"/>
-      <inertia ixx="1e-6" ixy="0" ixz="0" iyy="1e-6" iyz="0" izz="1e-6" />
-    </inertial>
-  </link>
+<!-- ============ imu_link xacro:macro ========================= -->
+  <xacro:macro name="imu_sensor">
+    <joint name="imu_joint" type="fixed">
+      <parent link="base_link"/>
+      <child link="imu_link"/>
+      <origin xyz="0.08 -0.06 -0.01" rpy="0 0 0"/>
+    </joint>
+    <link name="imu_link">
+      <visual>
+        <origin xyz="0 0 0" rpy="0 0 0"/>
+        <geometry>
+          <box size="0.003 0.010 0.015"/>
+        </geometry>
+        <material name="cyan"/>
+      </visual>
+    </link>
+  </xacro:macro>
+<!-- ============ imu_link xacro:if ========================= -->
+  <!-- if using a property (just inside this URDF file)-->
+  <!--xacro:if value="${imu == 'true'}"-->
+  <!--xacro:if value="${imu}"-->
+  <!-- if using an argument (call from outside)-->
+  <xacro:if value="$(arg imu)">
+    <xacro:imu_sensor/>
+  </xacro:if>
+<!-- ============ Distance sensor ====================== -->
+  <xacro:macro name="distance_sensor">
+  <!-- JOINT distance_sensor to base_link -->
+    <joint name="distance_sensor_joint" type="fixed">
+      <axis xyz="0 1 0" />
+      <origin xyz="0.085 0 0.025" rpy="0 0 0"/>
+      <parent link="base_link"/>
+      <child link="distance_sensor"/>
+    </joint>
+  <!-- Distance Sensor -->
+    <link name="distance_sensor">
+      <visual>
+        <origin xyz="0 0 0" rpy="1.57 0 1.57"/>
+        <geometry>
+          <mesh filename="package://gopigo3_description/meshes/sensors/IR_Sensor_Sharp_GP2Y_solid.stl" scale="0.001 0.001 0.001"/>
+        </geometry>
+        <material name="red"/>
+      </visual>
+    </link>
+  </xacro:macro>
+  <xacro:if value="$(arg distance)">
+    <xacro:distance_sensor/>
+  </xacro:if>
+<!-- ============ base_scan ======================== -->
+  <xacro:macro name="lds_sensor">
+    <joint name="scan_joint" type="fixed">
+      <parent link="base_link"/>
+      <child link="base_scan"/>
+      <origin xyz="-0.02 0 0.105" rpy="0 0 -1.6"/>
+      <!--LDS** origin xyz="-0.02 0 0.07" rpy="0 0 -1.6"/-->
+    </joint>
+    <link name="base_scan">
+      <visual>
+        <origin xyz="0 0 0.0" rpy="0 0 0"/>
+        <geometry>
+          <mesh filename="package://gopigo3_description/meshes/sensors/X4.stl" scale="0.001 0.001 0.001"/>
+          <!--LDS** mesh filename="package://gopigo3_description/meshes/sensors/lds.stl" scale="0.001 0.001 0.001"/-->
+        </geometry>
+        <material name="orange"/>
+      </visual>
+  <!-- **** base_scan COLLISION & INERTIA **** -->
+      <collision>
+        <origin xyz="0.015 0 -0.0065" rpy="0 0 0"/>
+        <geometry>
+          <cylinder length="0.05" radius="0.035"/>
+        </geometry>
+      </collision>
+      <inertial>
+        <mass value="0.178" />
+        <origin xyz="0 0 0" />
+        <inertia ixx="1.10e-04" ixy="-1.56e-04" ixz="-3.12e-04"
+                 iyy="1.85e-04" iyz="-2.23e-04"
+                 izz="2.21e-04" />
+      </inertial>
+    </link>
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