Commit message: Several bugfixes and tweaks in XACRO files to make the GoPiGo3 model behave more realistic in Gazebo simulation

File: gopigo3_description/urdf/gopigo3.gazebo.xacro (robot description, xacro)
@@ -10,10 +10,10 @@
 <!-- Left wheel mechanical properties -->
   <gazebo reference="wheel_left_link">
-    <mu1>0.1</mu1>
-    <mu2>0.1</mu2>
+    <mu1>0.5</mu1>
+    <mu2>0.5</mu2>
     <kp>500000.0</kp>
     <kd>10.0</kd>
     <minDepth>0.001</minDepth>
-    <maxVel>0.1</maxVel>
+    <maxVel>0.5</maxVel>
     <fdir1>1 0 0</fdir1>
     <material>Gazebo/FlatBlack</material>
@@ -21,10 +21,10 @@
 <!-- Right wheel mechanical properties -->
   <gazebo reference="wheel_right_link">
-    <mu1>0.1</mu1>
-    <mu2>0.1</mu2>
+    <mu1>0.5</mu1>
+    <mu2>0.5</mu2>
     <kp>500000.0</kp>
     <kd>10.0</kd>
     <minDepth>0.001</minDepth>
-    <maxVel>0.1</maxVel>
+    <maxVel>0.5</maxVel>
     <fdir1>1 0 0</fdir1>
     <material>Gazebo/FlatBlack</material>
@@ -32,10 +32,10 @@
 <!-- Caster back mechanical properties -->
   <gazebo reference="caster_back_link">
-    <mu1>0.1</mu1>
-    <mu2>0.1</mu2>
+    <mu1>0.001</mu1>
+    <mu2>0.001</mu2>
     <kp>1000000.0</kp>
     <kd>100.0</kd>
     <minDepth>0.001</minDepth>
-    <maxVel>1.0</maxVel>
+    <maxVel>10.0</maxVel>
     <material>Gazebo/FlatBlack</material>
   </gazebo>
@@ -144,5 +144,5 @@
       <pose>0 0 0 0 0 0</pose>
       <visualize>$(arg laser_visual)</visualize>
-      <update_rate>5</update_rate>
+      <update_rate>10</update_rate>
       <ray>
         <scan>
@@ -150,6 +150,6 @@
             <!--samples>360</samples>
             <resolution>1</resolution-->
-            <samples>720</samples>
-            <resolution>0.5</resolution>
+            <samples>500</samples>
+            <resolution>0.72</resolution>
             <min_angle>0.0</min_angle>
             <max_angle>6.28319</max_angle>
@@ -216,5 +216,5 @@
    </gazebo>
 <!-- 2D Camera controller -->
-  <gazebo reference="camera">
+  <gazebo reference="camera_rgb_frame">
     <sensor type="camera" name="camera1">
       <always_on>true</always_on>
@@ -238,5 +238,5 @@
         <imageTopicName>image_raw</imageTopicName>
         <cameraInfoTopicName>camera_info</cameraInfoTopicName>
-        <frameName>camera</frameName>
+        <frameName>camera_rgb_frame</frameName>
         <hackBaseline>0.07</hackBaseline>
         <distortionK1>0.0</distortionK1>

File: gopigo3_description/urdf/gopigo3.urdf.xacro (robot description, xacro)
@@ -23,16 +23,25 @@
   <!-- **** 'base_link' COLLISION & INERTIA **** -->
     <collision>
-      <origin xyz="-0.032 0 0.070" rpy="0 0 0"/>
-      <geometry>
-        <box size="0.21 0.105 0.11"/>
-      </geometry>
-    </collision>
-    <inertial>
-      <origin xyz="0 0 0" rpy="0 0 0"/>
+      <origin xyz="-0.038 0 -0.015" rpy="0 0 0"/>
+      <geometry>
+        <box size="0.245 0.088 0.07"/>
+      </geometry>
+    </collision>
+    <inertial>
+      <origin xyz="-0.02 0 0" rpy="0 0 0"/>
       <mass value="0.534"/>
-      <inertia ixx="1.03e-03" ixy="-1.54e-03" ixz="-2.94e-03"
+      <!-- <inertia ixx="1.03e-03" ixy="-1.54e-03" ixz="-2.94e-03"
                iyy="2.50e-03" iyz="-3.08e-03"
+               izz="2.45e-03" /> -->
+      <inertia ixx="1.0e-03" ixy="0" ixz="0"
+               iyy="1.0e-03" iyz="0"
                izz="2.45e-03" />
     </inertial>
+    <!-- <visual>
+      <origin xyz="-0.038 0 -0.015" rpy="0 0 0"/>
+      <geometry>
+        <box size="0.245 0.088 0.07"/>
+      </geometry>
+    </visual> -->
   </link>
 <!-- ============  'base_link_cad' is the solid model of robot body ====== -->
@@ -41,10 +50,10 @@
     <child link="base_link_cad"/>
     <!-- CAD of body of GoPiGo3 has its reference coordinate system at the center of the wheels shaft -->
-    <origin xyz="0 0 0.033" rpy="0 0 -4.71"/>
+    <origin xyz="-0.02 0 0.033" rpy="0 0 -4.71"/>
   </joint>
   <link name="base_link_cad">
     <visual>
       <!-- Decentering of the CAD model coordinate system-->
-      <origin xyz="0.024 0.097 -0.038" rpy="0 0 0"/>
+      <origin xyz="0.03 0.097 -0.038" rpy="0 0 0"/>
       <geometry>
         <mesh filename="package://gopigo3_description/meshes/GoPiGo3_Body.stl" scale="${CADscale} ${CADscale} ${CADscale}"/>
@@ -64,8 +73,12 @@
   <link name="wheel_left_link">
     <visual>
+      <!-- <origin xyz="0 0 0" rpy="0 1.57 0"/>
+      <geometry>
+        <cylinder length="0.026" radius="0.033"/>
+      </geometry>     -->
       <!-- Decentering of wheel CAD model coordinate system-->
-      <origin xyz="-0.195 -0.173 -0.029" rpy="0 0 0"/>
-      <geometry>
-        <mesh filename="package://gopigo3_description/meshes/GoPiGo3_Wheel.stl" scale="0.001 0.001 0.001"/>
+      <origin xyz="-0.22581 -0.200334 -0.033582" rpy="0 0 0"/>
+      <geometry>
+        <mesh filename="package://gopigo3_description/meshes/GoPiGo3_Wheel.stl" scale="0.001158 0.001158 0.001158"/>
       </geometry>
       <material name="black"/>
@@ -73,5 +86,5 @@
   <!-- **** 'wheel_left' COLLISION & INERTIA **** -->
     <collision>
-      <origin xyz="0 0 0" rpy="0 0 0"/>
+      <origin xyz="0 0 0" rpy="0 1.57 0"/>
       <geometry>
         <cylinder length="0.026" radius="0.033"/>
@@ -96,8 +109,12 @@
   <link name="wheel_right_link">
     <visual>
+      <!-- <origin xyz="0 0 0" rpy="0 1.57 0"/>
+      <geometry>
+        <cylinder length="0.026" radius="0.033"/>
+      </geometry> -->
       <!-- Decentering of wheel CAD model coordinate system-->
-      <origin xyz="-0.195 -0.173 -0.029" rpy="0 0 0"/>
-      <geometry>
-        <mesh filename="package://gopigo3_description/meshes/GoPiGo3_Wheel.stl" scale="0.001 0.001 0.001"/>
+      <origin xyz="-0.22581 -0.200334 -0.033582" rpy="0 0 0"/>
+      <geometry>
+        <mesh filename="package://gopigo3_description/meshes/GoPiGo3_Wheel.stl" scale="0.001158 0.001158 0.001158"/>
       </geometry>
       <material name="black"/>
@@ -105,5 +122,5 @@
   <!-- **** 'wheel_right' COLLISION & INERTIA **** -->
     <collision>
-      <origin xyz="0 0 0" rpy="0 0 0"/>
+      <origin xyz="0 0 0" rpy="0 1.57 0"/>
       <geometry>
         <cylinder length="0.026" radius="0.033"/>
@@ -122,14 +139,20 @@
     <parent link="base_link"/>
     <child link="caster_back_link"/>
-    <origin xyz="-0.115 0 -0.075" rpy="0 0 0"/>
+    <origin xyz="-0.132 0 -0.075" rpy="0 0 0"/>
   </joint>
   <link name="caster_back_link">
   <!-- **** COLLISION & INERTIA **** -->
     <collision>
-      <origin xyz="0 0.001 0" rpy="0 0 0"/>
-      <geometry>
-        <box size="0.030 0.009 0.020"/>
-      </geometry>
-    </collision>
+      <origin xyz="0 0 0.01" rpy="1.57 0 0"/>
+      <geometry>
+        <cylinder length="0.009" radius="0.01"/>
+      </geometry>
+    </collision>
+    <!-- <visual>
+      <origin xyz="0 0 0.01" rpy="1.57 0 0"/>
+      <geometry>
+        <cylinder length="0.009" radius="0.01"/>
+      </geometry>
+    </visual> -->
     <inertial>
       <origin xyz="0 0 0" />
@@ -145,5 +168,5 @@
       <parent link="base_link"/>
       <child link="imu_link"/>
-      <origin xyz="0.08 -0.06 -0.01" rpy="0 0 0"/>
+      <origin xyz="0.06 -0.06 -0.01" rpy="0 0 0"/>
     </joint>
     <link name="imu_link">
@@ -170,5 +193,5 @@
     <joint name="distance_sensor_joint" type="fixed">
       <axis xyz="0 1 0" />
-      <origin xyz="0.085 0 0.025" rpy="0 0 0"/>
+      <origin xyz="0.065 0 0.025" rpy="0 0 0"/>
       <parent link="base_link"/>
       <child link="distance_sensor"/>
@@ -193,10 +216,10 @@
       <parent link="base_link"/>
       <child link="base_scan"/>
-      <origin xyz="-0.02 0 0.105" rpy="0 0 -1.6"/>
+      <origin xyz="-0.02 0 0.085" rpy="0 0 -1.57"/>
       <!--LDS** origin xyz="-0.02 0 0.07" rpy="0 0 -1.6"/-->
     </joint>
     <link name="base_scan">
       <visual>
-        <origin xyz="0 0 0.0" rpy="0 0 0"/>
+        <origin xyz="0 0 0.02" rpy="0 0 0"/>
         <geometry>
           <mesh filename="package://gopigo3_description/meshes/sensors/X4.stl" scale="0.001 0.001 0.001"/>
@@ -204,10 +227,14 @@
         </geometry>
         <material name="orange"/>
+        <!-- <origin xyz="0 0 -0.0215" rpy="0 0 0"/>
+        <geometry>
+          <cylinder length="0.055" radius="0.035"/>
+        </geometry> -->
       </visual>
   <!-- **** base_scan COLLISION & INERTIA **** -->
       <collision>
-        <origin xyz="0.015 0 -0.0065" rpy="0 0 0"/>
-        <geometry>
-          <cylinder length="0.05" radius="0.035"/>
+        <origin xyz="0 0 -0.0215" rpy="0 0 0"/>
+        <geometry>
+          <cylinder length="0.055" radius="0.035"/>
         </geometry>
       </collision>
@@ -237,5 +264,5 @@
     <!-- **** Pi Camera COLLISION & INERTIA **** -->
       <collision>
-        <origin xyz="0.005 0.011 0.013" rpy="0 0 0"/>
+        <origin xyz="0.005 0 0.013" rpy="0 0 0"/>
         <geometry>
           <box size="0.015 0.030 0.027"/>
@@ -247,5 +274,5 @@
   <!-- (JOINTS) Pi Camera -->
     <joint name="camera_joint" type="fixed">
-      <origin xyz="0.06 0 0.04" rpy="0 0 0"/>
+      <origin xyz="0.04 0 0.04" rpy="0 0 0"/>
       <parent link="base_link"/>
       <child link="camera_link"/>
