Commit message: Change wheel rotation direction in URDF
This is needed to go forward in response to a positive velocity command.

File: gopigo3_description/urdf/gopigo3.urdf.xacro (robot description, xacro)
@@ -69,5 +69,5 @@
     <!-- Tz = -(0.075 base_link cdg -0.033 wheel radius) = -0.042 -->
     <origin xyz="0 0.058 -0.042" rpy="0 0 1.57"/>
-    <axis xyz="-1 0 0"/>
+    <axis xyz="1 0 0"/>
   </joint>
   <link name="wheel_left_link">
@@ -105,5 +105,5 @@
     <origin xyz="0 -0.058 -0.042" rpy="0 0 -1.57"/>
     <!--axis xyz="0 0 1"/-->
-    <axis xyz="1 0 0"/>
+    <axis xyz="-1 0 0"/>
   </joint>
   <link name="wheel_right_link">
